File: ITC-1/ITC-1.sch (KiCad schematic (older format))
At the start: 23 parts, among them K1 кнопка, K2 кнопка, X1 крепеж, X2 крепеж

Commit message: расположено управление светодиодами
Parts:
- added C1, C2: Конденсатор_керамический, N_RLC:Конденсатор_SMD_0603_pnp, symbol elements:Конденсатор_керамический
- added DA1, DA2: ОУ_LMx58, N_DD:SO-8, symbol elements:ОУ_LMx58
- added G1: стабилизатор_нерегулируемый_LM1117S33, N_VD_HL:Транзистор_NPN_SOT223_pnp, symbol elements:стабилизатор_нерегулируемый_LM1117S33
- added R1, R10, R11, R12, R13, R14, R15, R16, R17, R18, R19, R2, R20, R21, R22, R23, R24, R25, R26, R27, R28, R3, R4, R5, R6, R7, R8, R9: Резистор_0,065Вт, N_RLC:Резистор_SMD_0603_0,065_Вт_pnp, symbol elements:Резистор_0,065Вт
- added VT1, VT2: Транзистор_полевой_P-канал(IRLML2246TRPBF), N_VD_HL:Транзистор_IRLML6344TR_SOT-23, symbol elements:Транзистор_полевой_P-канал(IRLML2246TRPBF)
- added VT10, VT11, VT3, VT4, VT5, VT6, VT7, VT8, VT9: Транзистор_полевой_N-IRLML6344TR, N_VD_HL:Транзистор_IRLML6344TR_SOT-23, symbol elements:Транзистор_полевой_N-IRLML6344TR
- added XP1: Вилка_PLD6_ПРОГ_STM, N_X:Вилка_PLLD6_угловая_вертикальная, symbol elements:Вилка_PLD6_ПРОГ_STM
- added XP2: Клеммник_х2, N_X:Вилка_XH2.54-2_вертикальная, symbol elements:Клеммник_х2
- added XP3: Клеммник_х4, N_X:Вилка_XH2.54-4_вертикальная, symbol elements:Клеммник_х4
Connections:
- net GND: now reaches A1.1 (GND)
- net GND: now also A1.15 (GND), A1.38 (GND), A1.39 (GND), K1.2, K2.2, C1.2, C2.2, G1.1 (GND), R1.2, R15.2, R16.2, R2.2, R5.2, R6.2, R7.2, R8.2, R9.2, VT10.2, VT11.2, VT3.2, VT4.2, VT5.2, VT6.2, VT7.2, VT8.2, VT9.2, XP1.6 (GND)
- net LED_5: now reaches A1.10 (IO25)
- net LED_5: now also R7.1, VT7.1
- net LED_6: now reaches A1.11 (IO26)
- net LED_6: now also R8.1, VT8.1
- net LED_7: now reaches A1.12 (IO27)
- net LED_7: now also R9.1, VT9.1
- net LED_8: now reaches A1.13 (IO14)
- net LED_8: now also R15.1, VT10.1
- net LED_9: now reaches A1.16 (IO13)
- net LED_9: now also R16.1, VT11.1
- net 3V3: now reaches A1.2 (3V3)
- net 3V3: now also C2.1, G1.2 (3В3), R19.1, R20.1, R23.1, R26.1, R27.2, R28.2, VT1.2, VT2.2, XP1.2 (3V)
- net LED_GREEN: now reaches A1.23 (IO15)
- net LED_GREEN: now also R28.1, VT2.1
- net LED_RED: now reaches A1.24 (IO2)
- net LED_RED: now also R27.1, VT1.1
- net BOOT_SEL: now reaches A1.25 (IO(ноль)_BOOT)
- net BOOT_SEL: now also R23.2, R24.1
- net BUTT_1: now reaches A1.26 (IO4)
- net BUTT_1: now also R20.2, R21.1
- net BUTT_2: now reaches A1.27 (IO16)
- net BUTT_2: now also R19.2, R22.1
- net EN_RESET: now reaches A1.3 (EN)
- net EN_RESET: now also R25.1, R26.2
- net BOOT_UART_RX: now reaches A1.34 (RXD0)
- net BOOT_UART_RX: now also XP1.3 (SLK)
- net BOOT_UART_TX: now reaches A1.35 (TXD0)
- net BOOT_UART_TX: now also XP1.4 (DIO)
- net LED_1: now reaches A1.6 (IO34)
- net LED_1: now also R1.1, VT3.1
- net LED_2: now reaches A1.7 (IO35)
- net LED_2: now also R2.1, VT4.1
- net LED_3: now reaches A1.8 (IO32)
- net LED_3: now also R5.1, VT5.1
- net LED_4: now reaches A1.9 (IO33)
- net LED_4: now also R6.1, VT6.1
- net 3V3-RED: now reaches HL1.1
- net 3V3-RED: now also HL11.1, HL13.1, HL15.1, HL17.1, HL3.1, HL5.1, HL7.1, HL9.1, VT1.3
- net at HL1.2: now also HL2.2, R3.1
- net 3V3-GREEN: now reaches HL2.1
- net 3V3-GREEN: now also HL10.1, HL12.1, HL14.1, HL16.1, HL18.1, HL4.1, HL6.1, HL8.1, VT2.3
- net at K1.1: now also R21.2
- net at K2.1: now also R22.2
- net at HL3.2: now also HL4.2, R4.1
- net at HL5.2: now also HL6.2, R10.1
- net at HL7.2: now also HL8.2, R11.1
- net at HL9.2: now also HL10.2, R12.1
- net at HL11.2: now also HL12.2, R13.1
- net at HL13.2: now also HL14.2, R14.1
- net at HL15.2: now also HL16.2, R17.1
- net at HL17.2: now also HL18.2, R18.1
- new net: R24.2, XP1.1 (mode)
- new net: R25.2, XP1.5 (RST)
- new net: R3.2, VT3.3
- new net: R4.2, VT4.3
- new net: R10.2, VT5.3
- new net: R11.2, VT6.3
- new net: R12.2, VT7.3
- new net: R13.2, VT8.3
- new net: R14.2, VT9.3
- new net: R17.2, VT10.3
- new net: R18.2, VT11.3
- new net 1-LION: XP3.4
- new net 2-LION: XP3.3
- new net 3-LION: XP3.2
- new net 4-LION: C1.1, G1.3 (4...15_В), XP3.1
- new net CHARGE: XP2.1
- new net PWR-GND: XP2.2
- no-connect marks 0 -> 6
Other:
- moved on the sheet: HL1, HL10, HL11, HL12, HL13, HL14, HL15, HL16, HL17, HL18, HL2, HL3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

Commit message: заменены разъемы, исключены ОУ, определена распиновка и упр. транзистор
Parts:
- removed DA1, DA2: ОУ_LMx58, N_DD:SO-8, symbol elements:ОУ_LMx58
- removed XP2: Клеммник_х2, N_X:Вилка_XH2.54-2_вертикальная, symbol elements:Клеммник_х2
- removed XP3: Клеммник_х4, N_X:Вилка_XH2.54-4_вертикальная, symbol elements:Клеммник_х4
- added R29, R30, R31: Резистор_0,065Вт, N_RLC:Резистор_SMD_0603_0,065_Вт_pnp, symbol elements:Резистор_0,065Вт
- added VD1: Диод_шоттки, N_VD_HL:Диод_SMB_pnp, symbol elements:Диод_шоттки
- added VT12: Транзистор_полевой_N-IRLML6344TR, N_VD_HL:Транзистор_IRLML6344TR_SOT-23, symbol elements:Транзистор_полевой_N-IRLML6344TR
- added VT13: Транзистор_NPN_1Б-2(4)К-3Э_0, N_VD_HL:Транзистор_NPN_SOT223_pnp, symbol elements:Транзистор_NPN_1Б-2(4)К-3Э_0
- added XP4, XP5: Вилка_PLS6, N_X:Вилка_PLD6_вертикальная, symbol elements:Вилка_PLS6
Connections:
- net 1-LION: now also XP5.4
- net 2-LION: now also XP5.3
- net 3-LION: now also XP5.2
- net 4-LION: now also R31.2, VD1.2, XP4.1, XP5.1
- net GND: now also R30.2, VT12.2, VT13.3, XP5.5, XP5.6
- new net: R29.2, VT13.1
- new net BUTTON-LED: R31.1, VT12.3, XP4.3
- new net CHARGE-SENS: XP4.2
- new net LED-DRIVE: R30.1, VT12.1
- new net MOTOR-DRIVE: R29.1
- new net MOTOR-GND: VD1.1, VT13.2, VT13.4, XP4.5, XP4.6
- no-connect marks 6 -> 7
Other:
- note added: "требует подобрать транзистор \nи проверить, подходит ли он"
- moved on the sheet: HL10, HL11, HL12, HL13, HL14, HL15, HL16, HL17, HL18, HL5, HL6, HL7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
