File: ITC-1/ITC-1.sch (KiCad schematic (older format))
At the start: 83 parts, among them K1 кнопка, K2 кнопка, K3 кнопка, X1 крепеж, X2 крепеж, X3 крепеж, X4 крепеж, X5 Вилка_PLS6, X6 Вилка_PLS4, X7 Check_point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

Commit message: ITC-1-1 исправлен проект
добавлены стабилизаторы на DIN и LI4, усилены дорожки, фаски с двух сторон
Parts:
- removed R42: Резистор_0,065Вт, N_RLC:Резистор_SMD_0603_0,065_Вт_pnp, symbol elements:Резистор_0,065Вт
- added R31: Резистор_0,065Вт, N_RLC:Резистор_SMD_0603_0,065_Вт_pnp, symbol elements:Резистор_0,065Вт
- added VD2, VD3: Стабилитрон_1N5352BRLG_вертикальный, N_VD_HL:SOD-80, symbol elements_2020:Стабилитрон_1N5352BRLG_вертикальный
- G1: symbol elements:стабилизатор_нерегулируемый_LM1117S33 -> elements:стабилизатор_нерегулируемый_LM1117S33-SOT223
Connections:
- net 3V3: now also G1.4 (BOT)
- net 4-LION: now also R31.1
- net CHARGE-SENS: now also VD2.2
- net GND: now also X4.1, VD2.1, VD3.1
- net MOTOR-GND: now also X3.1
- new net: R31.2, VD3.2
Other:
- moved on the sheet: C1, C2, C3, C7, G2, R32

Commit message: на esp32 убраны запрещенные площадки, сформированы gerber-файлы
Parts:
- A1: footprint N_A:ESP32_WROOM32_pnp -> N_A:ESP32_WROOM32_pnp_noSD; symbol modules:модуль_esp32_wroom_32_SMD -> modules:модуль_esp32_wroom_32_SMD_noSD
Connections:
- no-connect marks 8 -> 5
Changed lines of the file:
@@
 $EndDescr
 $Comp
-L modules:модуль_esp32_wroom_32_SMD A1
+L modules:модуль_esp32_wroom_32_SMD_noSD A1
 U 1 1 609973EE
 P 2200 2000
 F 0 "A1" H 3725 2265 50  0000 C CNN
 F 1 "модуль_esp32_wroom_32_SMD" H 3725 2174 50  0000 C CNN
-F 2 "N_A:ESP32_WROOM32_pnp" H 2200 2000 50  0001 C CNN
+F 2 "N_A:ESP32_WROOM32_pnp_noSD" H 2200 2000 50  0001 C CNN
 F 3 "" H 2200 2000 50  0001 C CNN
 F 4 "не заказывал, есть в наличии" H 2200 2000 50  0001 C CNN "LINK"
@@
 Text Label 1500 3350 0    50   ~ 0
 LED_1
-NoConn ~ 2000 3950
-NoConn ~ 3250 4250
-NoConn ~ 3400 4250
 Text Label 6250 2450 2    50   ~ 0
 BOOT_UART_TX
@@
 Entry Wire Line
 	6400 3950 6500 4050
-Entry Wire Line
-	1250 3100 1350 3200
-Wire Wire Line
-	1350 3200 2000 3200
 Text Label 1500 3500 0    50   ~ 0
 LED_2
@@
 Wire Wire Line
 	3750 1000 3750 1250
+Text Label 3750 1250 2    50   ~ 0
+MOTOR-GND
 Wire Bus Line
 	14500 1500 14500 4750
@@
 Wire Bus Line
 	1250 1500 1250 11650
-Text Label 3750 1250 2    50   ~ 0
-MOTOR-GND
 $EndSCHEMATC

Commit message: обновлена номенклатура для заказа ПКИ
Parts:
- A1, K1, K2, K3: ORDER (none) -> не заказывал, есть в наличии
- C1: INFO (none) -> 10 мкФ/25 В; LINK https://www.chipdip.ru/product/grm188r71e105ka12d -> https://www.chipdip.ru/product/grm21br61e106ka73l; ORDER (none) -> 10
- C2, C3, C7: INFO (none) -> 10 мкФ/6,3 В; ORDER (none) -> 10
- C4, C5, C6: INFO (none) -> 1 мкФ/25 В; ORDER (none) -> 10
- D1, D2, X1, X2, X3, X4, X5, X6, X7, X8, X9: ORDER (none) -> -
- G1: LINK https://www.chipdip.ru/product/lm1117gs-3.3 -> https://www.chipdip.ru/product/ncp1117st33t3g-2; ORDER (none) -> 4
- G2: ORDER (none) -> 3
- HL1, HL2, HL3, HL4, HL5, HL6, HL7, HL8, HL9, VT10, VT11, VT3, VT4, VT5, VT6, VT7, VT8, VT9: ORDER (none) -> 30
- R1, R15, R16, R2, R20, R23, R26, R27, R28, R32, R37, R38, R39, R40, R41, R5, R6, R7, R8, R9: INFO (none) -> 10 кОм; LINK https://www.chipdip.ru/product0/65097 -> https://www.chipdip.ru/product0/9000079736; ORDER (none) -> 60
- R10, R11, R12, R13, R14, R17, R18, R21, R22, R3, R30, R4: INFO (none) -> 240 Ом; ORDER (none) -> 40
- R19: INFO (none) -> 30 кОм; LINK https://www.chipdip.ru/product0/20824 -> https://www.chipdip.ru/product0/9000079747; ORDER (none) -> 20
- R24: INFO (none) -> 51 кОм; LINK https://www.chipdip.ru/product0/469851073 -> https://www.chipdip.ru/product0/9000079753; ORDER (none) -> 20
- R25, R29: INFO (none) -> 1,3 кОм; LINK https://www.chipdip.ru/product0/10149 -> https://www.chipdip.ru/product0/43144; ORDER (none) -> 20; Номинал 1 кОм -> 1,3 кОм
- R31: INFO (none) -> 39 Ом; LINK https://www.chipdip.ru/product0/65097 -> https://www.chipdip.ru/product0/18162; ORDER (none) -> 20
- R33: INFO (none) -> 68 кОм; LINK https://www.chipdip.ru/product0/36049 -> https://www.chipdip.ru/product0/9000079756; ORDER (none) -> 20
- VD2: LINK https://www.chipdip.ru/product/1n5352brlg-2 -> https://www.chipdip.ru/product/bzv55c2v7; ORDER (none) -> 4
- VD3: LINK https://www.chipdip.ru/product/1n5352brlg-2 -> https://www.chipdip.ru/product/bzv55c18; ORDER (none) -> 4
- VT1, VT2: ORDER (none) -> 8
- VT12: LINK (none) -> https://www.chipdip.ru/product/std17nf03lt4-2; ORDER (none) -> 4
